File: RF-AMP-QSK-SWITCH_V1.kicad_pcb (KiCad board)
At the start: 2 copper layers, 100 x 160 mm, 193 parts, among them J1 TRX, J2 AMP_IN, J3 ANT, J4 AMP_OUT, Q1 BCP56, Q10 PBHV2160Z, Q11 BC857, Q13 MMBTA92, Q14 BC817, Q15 MMBTA92, Q16 MMBTA92, Q17 MMBTA92, Q18 MMBTA42, Q19 BC857, Q2 STN9260, Q21 MMBTA92, Q22 MMBTA92, Q23 BC817, Q24 BC857, Q25 BC817, Q26 BC857, Q27 BC817, Q28 BC817, Q3 STN9260, Q4 BC817, Q5 STN9260, Q6 STN9260, Q7 STN9260, Q8 STN9260, Q9 STN9260, U1 LM2576S-ADJ, U2 L78L12_SOT89, U3 LT1963AEQ

Commit message: initial commit
Parts:
- removed L5: 820n, RF-AMP-QSK-SWITCH_V1:Air_Coil_1
- added L8: 820n, RF-AMP-QSK-SWITCH_V1:Coilcraft_Maxi_Spring, F.Cu at (141.5, 50.8)
- D16: value TX -> POWER
- L1, L2, L3, L4, L6, L7: footprint RF-AMP-QSK-SWITCH_V1:Air_Coil_1 -> RF-AMP-QSK-SWITCH_V1:Coilcraft_Maxi_Spring
- R1: footprint Resistor_SMD:R_1210_3225Metric -> Resistor_SMD:R_1206_3216Metric
- moved D16 68.1 mm to (56.2, 137.5), turned to 270 degrees
- moved R41 64.8 mm to (57.2, 142.5), turned to 180 degrees
- moved D12 39.3 mm to (56.2, 134.5), turned to 90 degrees
- moved L6 38.4 mm to (111.2, 54.0)
- moved Q24 32.0 mm to (61.0, 125.0), turned to 90 degrees
- moved L7 30.0 mm to (133.5, 68.8), turned to 0 degrees
- moved C10 29.5 mm to (126.5, 67.0), turned to 270 degrees
- moved C3 29.5 mm to (73.5, 67.0), turned to 270 degrees
- moved R34 28.0 mm to (56.2, 126.0), turned to 270 degrees
- moved R48 26.3 mm to (58.2, 126.0), turned to 90 degrees
- moved R35 25.1 mm to (55.0, 108.5), turned to 270 degrees
- moved Q23 23.7 mm to (64.5, 125.0), turned to 180 degrees
- moved R43 21.0 mm to (64.5, 122.2)
- moved R19 20.6 mm to (113.8, 106.2), turned to 90 degrees
- moved R36 20.6 mm to (55.0, 112.0), turned to 270 degrees
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- renumbered C16 to C15, C17 to C16, C18 to C17, C19 to C18, C20 to C19, C22 to C20, C23 to C21, C24 to C22, C25 to C23, C26 to C24, C28 to C25, C29 to C26, C30 to C27, C31 to C28, C32 to C29, C33 to C30, C34 to C31, C35 to C32, C37 to C33, C36 to C34, C38 to C35, C39 to C36, C40 to C37, C41 to C38, C42 to C39, C43 to C40, C44 to C41, C45 to C42, C46 to C43, C47 to C44, C48 to C45, C49 to C46, C50 to C47, C51 to C48, C52 to C49, C53 to C50, C54 to C51, C55 to C52, C56 to C53, C57 to C54, C58 to C55, C59 to C56, D12 to D11, D11 to D12, L9 to L10, L10 to L11, L8 to L9, REF** to MH1, REF** to MH2, Q13 to Q12, Q15 to Q13, Q16 to Q15, Q17 to Q16, Q21 to Q17, Q22 to Q18, Q18 to Q19, Q19 to Q20, Q23 to Q21, Q24 to Q22, Q25 to Q23, Q26 to Q24, Q27 to Q25, Q28 to Q26, R11 to R10, R12 to R11, R13 to R12, R14 to R13, R15 to R14, R22 to R15, R23 to R16, R25 to R18, R24 to R22, R29 to R23, R26 to R24, R27 to R25, R28 to R26, R38 to R27, R41 to R28, R30 to R29, R31 to R30, R33 to R31, R42 to R32, R35 to R33, R36 to R34, R39 to R35, R40 to R36, R43 to R37, R44 to R38, R45 to R39, R5 to R4, R46 to R40, R47 to R41, R48 to R42, R49 to R43, R50 to R44, R51 to R45, R52 to R46, R53 to R47, R54 to R48, R55 to R49, R4 to R5, R56 to R50, R57 to R51, R58 to R52, R59 to R53, R60 to R54, R7 to R6, R8 to R7, R9 to R8, R10 to R9
Connections:
- D12 pad 1: Net-(D11-Pad1) (its old number) -> Earth
- D12 pad 2: Earth -> Net-(D12-Pad2)
- D16 pad 1: Net-(D16-Pad1) -> Earth
- D16 pad 2: Earth -> Net-(D16-Pad2)
- L6 pad 1: VSW1 -> VSW3
- L6 pad 2: Net-(C13-Pad1) -> Net-(C8-Pad1)
- L7 pad 1: Net-(C11-Pad1) -> VSW1
- L7 pad 2: Earth -> Net-(C13-Pad1)
- R1 pad 2: Net-(C7-Pad2) -> Net-(L5-Pad1)
- R34 pad 2: Net-(D11-Pad1) (its old number) -> Net-(D12-Pad2)
- R41 pad 2: Net-(D16-Pad1) -> Net-(D16-Pad2)
Routing:
- net +12V: track 1.76 -> 132.0 mm, vias 0 -> 2
- net VN2: track 0.00 -> 96.9 mm
- net VN1_EN: track 0.00 -> 92.8 mm, vias 0 -> 2
- net VP: track 41.5 -> 108.7 mm, vias 2 -> 6
- net VSW5: track 0.00 -> 43.9 mm
- net VSW4: track 0.00 -> 43.5 mm
- net VSW2: track 0.00 -> 41.3 mm
- net VN2_EN: track 0.00 -> 26.2 mm
- net Net-(Q20-Pad3): track 0.00 -> 20.3 mm
- net Earth: track 9.10 -> 28.1 mm, vias 0 -> 10
- net VSW1_ON__: track 0.00 -> 17.4 mm
- net VSW1: track 22.4 -> 38.0 mm
- net VSW3: track 39.1 -> 51.9 mm
- net Net-(R46-Pad1): track 0.00 -> 12.5 mm
- net VSW1_ON_: track 10.2 -> 20.5 mm
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- added copper zone on F.Cu, net +12V
- added copper zone on F.Cu, net 13V8
- added copper zone on F.Cu, net 5V
- added copper zone on F.Cu, net Net-(C1-Pad1)
- added copper zone on F.Cu, net Net-(C1-Pad2)
- added copper zone on F.Cu, net Net-(C11-Pad1)
- added copper zone on F.Cu, net Net-(C11-Pad2)
- added copper zone on F.Cu, net Net-(C13-Pad1)
- added copper zone on F.Cu, net Net-(C13-Pad2)
- added copper zone on F.Cu, net Net-(C2-Pad1)
- added copper zone on F.Cu, net Net-(C2-Pad2)
- added copper zone on F.Cu, net Net-(C31-Pad2)
- added copper zone on F.Cu, net Net-(C5-Pad1)
- added copper zone on F.Cu, net Net-(C5-Pad2)
- added copper zone on F.Cu, net Net-(C7-Pad2)
- added copper zone on F.Cu, net Net-(C8-Pad1)
- added copper zone on F.Cu, net Net-(D15-Pad1)
- added copper zone on F.Cu, net VP

Commit message: final commit
Parts:
- added C10: 1n, Capacitor_SMD:C_1210_3225Metric, F.Cu at (88.8, 74.5)
- added C13: 1n, Capacitor_SMD:C_1210_3225Metric, F.Cu at (132.5, 82.5)
- added C6: 1p8, Capacitor_SMD:C_1210_3225Metric, F.Cu at (91.8, 47.8)
- added D5: MA4PK2001, RF-AMP-QSK-SWITCH_V1:MA4PK200x, F.Cu at (100.0, 68.0)
- added J5: Screw_Terminal_01x08, TerminalBlock_Phoenix:TerminalBlock_Phoenix_MPT-0,5-8-2.54_1x08_P2.54mm_Horizontal, F.Cu at (55.0, 152.8)
- added L5: 538n, RF-AMP-QSK-SWITCH_V1:Coilcraft_Maxi_Spring, F.Cu at (94.2, 69.2)
- added REF**: KiCad-Logo2_5mm_SilkScreen, Symbol:KiCad-Logo2_5mm_SilkScreen, F.Cu at (62.0, 149.8)
- D1, D2, D3: value MA4P506-1072T -> MA4P504-1072T
- L1, L2, L3, L4, L6, L7: value 820n -> 538n
- moved R41 13.3 mm to (61.0, 129.8)
- moved D17 2.00 mm to (56.2, 139.5), turned to 90 degrees
- turned C14 to 90 degrees
- turned C15 to 90 degrees
- renumbered C9 to C11, C10 to C12, C13 to C14, C14 to C15, C11 to C16, C12 to C17, C15 to C18, C16 to C19, C17 to C20, C18 to C21, C19 to C22, C20 to C23, C21 to C24, C22 to C25, C23 to C26, C24 to C27, C25 to C28, C26 to C29, C27 to C30, C28 to C31, C29 to C32, C30 to C33, C31 to C34, C32 to C35, C33 to C36, C34 to C37, C35 to C38, C36 to C39, C37 to C40, C38 to C41, C39 to C42, C40 to C43, C41 to C44, C42 to C45, C43 to C46, C44 to C47, C45 to C48, C46 to C49, C47 to C50, C48 to C51, C49 to C52, C50 to C53, C51 to C54, C52 to C55, C53 to C56, C54 to C57, C55 to C58, C56 to C59, C6 to C7, C7 to C8, C8 to C9, D9 to D10, D10 to D11, D11 to D12, D12 to D13, D13 to D14, D14 to D15, D15 to D16, D16 to D17, D17 to D18, D18 to D19, D19 to D20, D20 to D21, D21 to D22, D22 to D23, D23 to D24, D24 to D25, D25 to D26, D26 to D27, D27 to D28, D28 to D29, D29 to D30, D30 to D31, D31 to D32, D32 to D33, D33 to D34, D34 to D35, D35 to D36, D36 to D37, D37 to D38, D5 to D6, D6 to D7, D7 to D8, D8 to D9
Connections:
- net 5V renamed +5V
- net VN1_EN renamed VN1_ON
- net VN2_EN renamed VN2_ON
- net VSW1_ON_ renamed VSW1_EN_
- C14 pad 1: Net-(C13-Pad1) -> Net-(C13-Pad2)
- C14 pad 2: Net-(C13-Pad2) -> Net-(C14-Pad2)
- C15 pad 1: Net-(C13-Pad1) -> Net-(C13-Pad2)
- C15 pad 2: Net-(C13-Pad2) -> Net-(C14-Pad2)
- C18 pad 2: VSW1_ON -> VSW1_EN
- C23 pad 2: VSW2_ON -> VSW2_EN
- C8 pad 2: Net-(C7-Pad2) -> Net-(C8-Pad2)
- D3 pad 1: Net-(C7-Pad2) -> Net-(C8-Pad2)
- D7 pad 2: Net-(C13-Pad1) -> Net-(C14-Pad2)
- L7 pad 2: Net-(C13-Pad1) -> Net-(C14-Pad2)
- R1 pad 2: Net-(L5-Pad1) -> Net-(C8-Pad2)
- R19 pad 2: VSW1_EN -> VSW1_ON
- R20 pad 1: VSW1_EN -> VSW1_ON
- R21 pad 2: VSW2_ON -> VSW2_EN
- R27 pad 2: VSW1_ON__ -> VSW1_EN__
- R35 pad 2: VSW2_EN -> VSW2_ON
- R36 pad 1: VSW2_EN -> VSW2_ON
- R6 pad 2: VSW1_ON -> VSW1_EN
Routing:
- net VSW1_ON: track 1.84 -> 91.5 mm, vias 0 -> 1
- net VSW1_EN: track 3.40 -> 69.6 mm
- net VSW2_ON: track 2.00 -> 56.3 mm, vias 0 -> 1
- net VP: track 108.7 -> 158.5 mm, vias 6 -> 5
- net +12V: track 132.0 -> 181.0 mm, vias 2 -> 3
- net 13V8: track 0.00 -> 47.3 mm, vias 0 -> 1
- net VSW2_EN: track 3.38 -> 44.8 mm
- net +5V: track 0.00 -> 18.9 mm, vias 0 -> 1
- net VN1_ON: track 92.8 -> 77.4 mm
- net Net-(D17-Pad2): track 2.49 -> 9.53 mm
- net VSW3: track 51.9 -> 56.0 mm
- net VSW1: track 38.0 -> 41.7 mm
- net VSW2: track 41.3 -> 44.8 mm
- net VSW5: track 43.9 -> 44.7 mm
- net Earth: track 28.1 -> 27.5 mm, vias 10 -> 225
- added copper zone on F.Cu, net Net-(C14-Pad2)
- added copper zone on F.Cu, net Net-(C8-Pad2)
- removed copper zone on F.Cu, net Net-(C13-Pad1)
- removed copper zone on F.Cu, net Net-(C16-Pad2)
- removed copper zone on F.Cu, net Net-(C7-Pad2)
Other:
- net class HV added: clearance 1, trace_width 0.25, via_dia 0.8, via_drill 0.4
- board text added: "RF-AMP-QSK-SWITCH_V1 HB9GKW"
- board text added: "TX"
- board text added: "VN"

Commit message: Revision1
Parts:
- C33, C59: value 470n -> 100n
- C36, C41, C42, C43, C44, C48, C49, C50, C51, C52, C53, C54, C55, C56: value 100n -> 1n
- C45: value 82n -> 470p
- L11: value 10u -> 68u
- Q25, Q26: value BC817 -> BSS138
- R14: value 1R5 -> 1
- R39: value 1M -> 100k
- R44: value 470k -> 100k
- R50: value 33 -> 0
- R52: value 3R3 -> 1k8
- R53: value 3R3 -> 3k3
